File: remoticon_badge.kicad_pcb (KiCad board)
At the start: 2 copper layers, 71.1 x 116.8 mm, 930 parts, among them CON1 AVR-ISP-6, IC1 IC1, J1 Conn_02x16_Odd_Even, J2 Conn_02x12_Odd_Even, P1 CONN_01X01, P2 CONN_01X01, P3 CONN_01X01, P4 CONN_01X01, P5 CONN_01X01

Commit message: remove the coppor zone from the SMD challenge for better "After Dark" look
Routing:
- net GND: track 21.7 -> 60.6 mm, vias 3 -> 4
- removed copper zone on F.Cu, net GND
